Commit message: added driff drive plugin

File: description/gazebo.xacro (robot description, xacro)
@@ -10,8 +10,26 @@
         <material>Gazebo/Blue</material>
     </gazebo>
-    <gazebo reference="castor">
+    <gazebo reference="caster">
         <material>Gazebo/Blue</material>
         <mu1 value="0.001"/>
         <mu2 value="0.001"/>
     </gazebo>
+    <gazebo>
+        <plugin name='diff_drive' filename='libgazebo_ros_diff_drive.so'>
+            <!-- Wheel Information -->
+            <left_joint>left_wheel_joint</left_joint>
+            <right_joint>right_wheel_joint</right_joint>
+            <wheel_separation>0.35</wheel_separation>
+            <wheel_diameter>0.2</wheel_diameter>
+            <!-- Limits -->
+            <max_wheel_torque>5</max_wheel_torque>
+            <max_wheel_acceleration>2.0</max_wheel_acceleration>
+            <!-- Output -->
+            <odometry_frame>odom</odometry_frame>
+            <robot_base_frame>base_link</robot_base_frame>
+            <publish_odom>true</publish_odom>
+            <publish_odom_tf>true</publish_odom_tf>
+            <publish_wheel_tf>true</publish_wheel_tf>
+        </plugin>
+    </gazebo>
 </robot>

File: description/robot_core.urdf.xacro (robot description, xacro)
@@ -65,5 +65,5 @@
         <parent link="chassis"/>
         <child link="right_wheel"/>
-        <axis xyz="0.0 0.0 1.0"/>
+        <axis xyz="0.0 0.0 -1.0"/>
         <!-- <limit lower="0.0" upper="0.0" effort="0.0" velocity="0.0"/> -->
     </joint>

Commit message: added laser sensor

File: description/gazebo.xacro (robot description, xacro)
@@ -33,3 +33,30 @@
         </plugin>
     </gazebo>
+    <gazebo reference="laser">
+        <sensor name="laser" type="ray">
+            <pose> 0 0 0 0 0 0 </pose>
+            <visualize>true</visualize>
+            <update_rate>10</update_rate>
+            <ray>
+                <scan>
+                    <horizontal>
+                        <samples>360</samples>
+                        <min_angle>-3.14</min_angle>
+                        <max_angle>3.14</max_angle>
+                    </horizontal>
+                </scan>
+                <range>
+                    <min>0.4</min>
+                    <max>5</max>
+                </range>
+            </ray>
+            <plugin name="laser_controller" filename="libgazebo_ros_ray_sensor.so">
+                <ros>
+                    <argument>~/out:=scan</argument>
+                </ros>
+                <output_type>sensor_msgs/LaserScan</output_type> <!-- baad mai explain kar dunga-->
+                <frame_name>laser</frame_name>
+            </plugin>
+        </sensor>
+    </gazebo>
 </robot>

File: description/robot_core.urdf.xacro (robot description, xacro)
@@ -117,3 +117,33 @@
         </collision>
     </link>
+    <joint name="laser_joint" type="fixed">
+        <origin xyz="0.15 0.0 0.1" rpy="0.0 0.0 0.0"/>
+        <parent link="chassis"/>
+        <child link="laser"/>
+        <axis xyz="0.0 0.0 0.0"/>
+        <limit lower="0.0" upper="0.0" effort="0.0" velocity="0.0"/>
+    </joint>
+    <link name="laser">
+        <xacro:inertial_cylinder mass="0.1" length="0.03" radius="0.05">
+            <origin xyz="0.0 0 0.0" rpy="0 0 0"/>
+        </xacro:inertial_cylinder>
+        <visual name="">
+            <origin xyz="0.0 0.0 0.0" rpy="0.0 0.0 0.0"/>
+            <geometry>
+                <!-- <box size="0.1 0.1 0.03"/> -->
+                <cylinder radius="0.05" length="0.03"/>
+            </geometry>
+                <color rgba="1.0 0.0 0.0 0.0"/>
+            <material name="">
+                <color rgba="1.0 1.0 0.0 1.0"/>
+                <texture filename=""/>
+            </material>
+        </visual>
+        <collision>
+            <origin xyz="0.0 0.0 0.0" rpy="0.0 0.0 0.0"/>
+            <geometry>
+                <box size="0.1 0.1 0.03"/>
+            </geometry>
+        </collision>
+    </link>
 </robot>
